Commit message: change lidar link  position

File: src/module2/diffrobot_description/urdf/diffrobot.xacro (robot description, xacro)
@@ -169,5 +169,6 @@
     </link>
     <joint name="laser_data_joint" type="fixed">
-        <origin xyz="0.0 0.0 0.0" rpy="0.0 -1.5708 -1.5708"/>
+        <!-- <origin xyz="0.20 0.0 0.13" rpy="0.0 -1.5708 -1.5708"/> -->
+        <origin xyz="0.20 0.0 0.13" rpy="0.0 0.0 0.0"/>
         <parent link="lidar_link"/>
         <child link="laser"/>

Commit message: lidar link

File: src/module2/diffrobot_description/urdf/diffrobot.xacro (robot description, xacro)
@@ -170,5 +170,5 @@
     <joint name="laser_data_joint" type="fixed">
         <!-- <origin xyz="0.20 0.0 0.13" rpy="0.0 -1.5708 -1.5708"/> -->
-        <origin xyz="0.20 0.0 0.13" rpy="0.0 0.0 0.0"/>
+        <origin xyz="0.0 0.0 0.0" rpy="0.0 0.0 0.0"/>
         <parent link="lidar_link"/>
         <child link="laser"/>

Commit message: lid pos

File: src/module2/diffrobot_description/urdf/diffrobot.xacro (robot description, xacro)
@@ -170,5 +170,5 @@
     <joint name="laser_data_joint" type="fixed">
         <!-- <origin xyz="0.20 0.0 0.13" rpy="0.0 -1.5708 -1.5708"/> -->
-        <origin xyz="0.0 0.0 0.0" rpy="0.0 0.0 0.0"/>
+        <origin xyz="0.20 0.0 0.13" rpy="0.0 0.0 0.0"/>
         <parent link="lidar_link"/>
         <child link="laser"/>

Commit message: xacro

File: src/module2/diffrobot_description/urdf/diffrobot.xacro (robot description, xacro)
@@ -9,5 +9,5 @@
     <link name="base_link">
         <inertial>
-            <origin xyz="0.0 0.0 0.0" rpy="0.0 0.0 0.0"/>
+            <origin xyz="0.0 0.0 0.145" rpy="0.0 0.0 0.0"/>
             <mass value="15.0"/>
             <inertia ixx="0.0" ixy="0.0" ixz="0.0" iyy="0.0" iyz="0.0" izz="0.0"/>
@@ -170,5 +170,5 @@
     <joint name="laser_data_joint" type="fixed">
         <!-- <origin xyz="0.20 0.0 0.13" rpy="0.0 -1.5708 -1.5708"/> -->
-        <origin xyz="0.20 0.0 0.13" rpy="0.0 0.0 0.0"/>
+        <origin xyz="0.0 0.0 0.0" rpy="0.0 0.0 0.0"/>
         <parent link="lidar_link"/>
         <child link="laser"/>

Commit message: caster radius

File: src/module2/diffrobot_description/urdf/diffrobot.xacro (robot description, xacro)
@@ -89,5 +89,5 @@
             <origin xyz="0.0 0.0 0.0" rpy="0.0 0.0 0.0"/>
             <geometry>
-                <cylinder radius="0.0625" length="0.025"/>
+                <cylinder radius="0.08" length="0.025"/>
             </geometry>
             <material name="">
@@ -99,5 +99,5 @@
              <origin xyz="0.0 0.0 0.0" rpy="0.0 0.0 0.0"/>
             <geometry>
-                <cylinder radius="0.0625" length="0.025"/>
+                <cylinder radius="0.08" length="0.025"/>
             </geometry>
         </collision>
@@ -118,5 +118,5 @@
             <origin xyz="0.0 0.0 0.0" rpy="0.0 0.0 0.0"/>
             <geometry>
-                <cylinder radius="0.0625" length="0.025"/>
+                <cylinder radius="0.08" length="0.025"/>
             </geometry>
             <material name="">
@@ -128,5 +128,5 @@
            <origin xyz="0.0 0.0 0.0" rpy="0.0 0.0 0.0"/>
             <geometry>
-                <cylinder radius="0.0625" length="0.025"/>
+                <cylinder radius="0.08" length="0.025"/>
             </geometry>
         </collision>

Commit message: urdf file

File: src/module2/diffrobot_description/urdf/diffrobot.xacro (robot description, xacro)
@@ -3,13 +3,16 @@
     <xacro:include filename="$(find diffrobot_description)/urdf/diffrobot.gazebo"/>
     <link name="base_footprint"/>
-  <joint name="base_footprint_joint" type="fixed">
-      <parent link="base_footprint"/>
-      <child link="base_link"/>
-  </joint>
+    <joint name="base_footprint_joint" type="fixed">
+        <parent link="base_footprint"/>
+        <child link="base_link"/>
+    </joint>
     <link name="base_link">
         <inertial>
             <origin xyz="0.0 0.0 0.145" rpy="0.0 0.0 0.0"/>
             <mass value="15.0"/>
-            <inertia ixx="0.0" ixy="0.0" ixz="0.0" iyy="0.0" iyz="0.0" izz="0.0"/>
+            <inertia
+                ixx="0.1" ixy="0.0" ixz="0.0"
+                iyy="0.1" iyz="0.0"
+                izz="0.1"/>
         </inertial>
         <visual name="base_link_visual">
@@ -109,5 +112,5 @@
         <axis xyz="0.0 0.0 1.0"/>
     </joint>
- <link name="back_caster">
+    <link name="back_caster">
        <inertial>
             <origin xyz="0.0 0.0 0.0" rpy="0.0 0.0 0.0"/>
@@ -138,89 +141,35 @@
         <axis xyz="0.0 0.0 0.0"/>
     </joint>
-    <link name="lidar_link">
-        <inertial>
-            <origin xyz="0.0 0.0 0.0" rpy="0.0 0.0 0.0"/>
-            <mass value="0.1"/>
-            <inertia ixx="0.0" ixy="0.0" ixz="0.0" iyy="0.0" iyz="0.0" izz="0.0"/>
-        </inertial>
-        <visual name="lidar_link_visual">
+    <link name="laser">
+        <visual name="laser_visual">
             <origin xyz="0.0 0.0 0.0" rpy="0.0 0.0 0.0"/>
             <geometry>
-                <mesh filename="package://diffrobot_description/meshes/lidar_link.STL"/>
+                <box size="0.05 0.05 0.05"/>
             </geometry>
-            <material name="">
-                <color rgba="1.0 0.0 0.0 1.0"/>
-                <texture filename=""/>
-            </material>
         </visual>
-        <collision>
+        <collision name="laser_collision">
             <origin xyz="0.0 0.0 0.0" rpy="0.0 0.0 0.0"/>
             <geometry>
-                <box size="0.1 0.1 0.1"/>
+                <box size="0.05 0.05 0.05"/>
             </geometry>
         </collision>
     </link>
-    <joint name="lidar_joint" type="fixed">
-       <origin xyz="0.20 0.0 0.13" rpy="0.0 0.0 0.0"/>
+    <joint name="laser_data_joint" type="fixed">
+        <origin xyz="0.20 0.0 0.13" rpy="0.0 0.0 0.0"/>
         <parent link="base_link"/>
-        <child link="lidar_link"/>
-    </joint>
-    <link name="laser">
-    </link>
-    <joint name="laser_data_joint" type="fixed">
-        <!-- <origin xyz="0.20 0.0 0.13" rpy="0.0 -1.5708 -1.5708"/> -->
-        <origin xyz="0.0 0.0 0.0" rpy="0.0 0.0 0.0"/>
-        <parent link="lidar_link"/>
         <child link="laser"/>
     </joint>
-    <link name="gps_link">
-        <collision>
-        <origin xyz="0 0 0.1" rpy="0 0 0"/>
-        <geometry>
-            <box size="0.02 0.02 0.02"/>
-        </geometry>
-        </collision>
+    <link name="imu_link">
         <visual>
-        <origin xyz="0 0 0.1" rpy="0 0 0"/>
-        <geometry>
-            <box size="0.02 0.02 0.02"/>
-        </geometry>
-        <material name="orange"/>
+            <origin xyz="0 0 0" rpy="0 0 0"/>
+            <geometry>
+                <box size="0.03 0.1 0.03"/>
+            </geometry>
+            <material name="orange"/> <!-- Add this to fix the material warning -->
         </visual>
         <inertial>
-        <origin xyz="0 0 1" rpy="0 0 0"/>
-        <mass value="1"/>
-        <inertia
-            ixx="1.0" ixy="0.0" ixz="0.0"
-            iyy="1.0" iyz="0.0"
-            izz="1.0"/>
-        </inertial>
-    </link>
-    <joint name="gps_joint" type="fixed">
-        <origin xyz="0.0 0.0 0.0" rpy="0.0 0.0 0.0"/>
-        <parent link="base_link"/>
-        <child link="gps_link"/>
-    </joint>
-    <link name="imu_link">
-        <collision>
-        <origin xyz="0 0 0.1" rpy="0 0 0"/>
-        <geometry>
-            <box size="0.02 0.02 0.02"/>
-        </geometry>
-        </collision>
-        <visual>
-        <origin xyz="0.26 0 0" rpy="0 0 0"/>
-        <geometry>
-             <box size="0.03 0.1 0.03"/>
-        </geometry>
-        <material name="orange"/>
-        </visual>
-        <inertial>
-        <origin xyz="0 0 1" rpy="0 0 0"/>
-        <mass value="1"/>
-        <inertia
-            ixx="1.0" ixy="0.0" ixz="0.0"
-            iyy="1.0" iyz="0.0"
-            izz="1.0"/>
+            <origin xyz="0 0 0" rpy="0 0 0"/>
+            <mass value="0.1"/> <!-- Reduced mass (1kg is too heavy for an IMU) -->
+            <inertia ixx="1e-4" ixy="0.0" ixz="0.0" iyy="1e-4" iyz="0.0" izz="1e-4"/>
         </inertial>
     </link>

Commit message: update urdf

File: src/module2/diffrobot_description/urdf/diffrobot.xacro (robot description, xacro)
@@ -110,5 +110,4 @@
         <parent link="base_link"/>
         <child link="front_caster"/>
-        <axis xyz="0.0 0.0 1.0"/>
     </joint>
     <link name="back_caster">
@@ -139,5 +138,4 @@
         <parent link="base_link"/>
         <child link="back_caster"/>
-        <axis xyz="0.0 0.0 0.0"/>
     </joint>
     <link name="laser">

Commit message: urdf

File: src/module2/diffrobot_description/urdf/diffrobot.xacro (robot description, xacro)
@@ -3,5 +3,6 @@
     <xacro:include filename="$(find diffrobot_description)/urdf/diffrobot.gazebo"/>
     <link name="base_footprint"/>
-    <joint name="base_footprint_joint" type="fixed">
+    <joint name="robot_footprint_joint" type="fixed">
+        <origin xyz="0 0 0.0" rpy="0 0 0" />
         <parent link="base_footprint"/>
         <child link="base_link"/>
@@ -9,15 +10,12 @@
     <link name="base_link">
         <inertial>
-            <origin xyz="0.0 0.0 0.145" rpy="0.0 0.0 0.0"/>
-            <mass value="15.0"/>
-            <inertia
-                ixx="0.1" ixy="0.0" ixz="0.0"
-                iyy="0.1" iyz="0.0"
-                izz="0.1"/>
+            <origin xyz="0.0 0.0 0.0" rpy="0.0 0.0 0.0"/>
+            <mass value="5.0"/>
+            <inertia ixx="0.0" ixy="0.0" ixz="0.0" iyy="0.0" iyz="0.0" izz="0.0"/>
         </inertial>
         <visual name="base_link_visual">
             <origin xyz="0.0 0.0 0.0" rpy="0.0 0.0 0.0"/>
             <geometry>
-                <box size="0.52 0.52 0.155"/>
+                <box size="0.4 0.2 0.1"/>
             </geometry>
             <material name="">
@@ -29,18 +27,18 @@
             <origin xyz="0.0 0.0 0.0" rpy="0.0 0.0 0.0"/>
             <geometry>
-                <box size="0.52 0.52 0.155"/>
+                <box size="0.4 0.2 0.1"/>
             </geometry>
         </collision>
     </link>
     <link name="left_wheel">
-       <inertial>
-            <origin xyz="0.0 0.0 0.0" rpy="0.0 0.0 0.0"/>
-            <mass value="15.0"/>
+        <inertial>
+            <origin xyz="0.0 0.0 0.0" rpy="0.0 1.5707 1.5707"/>
+            <mass value="5.0"/>
             <inertia ixx="0.1" ixy="0.0" ixz="0.0" iyy="0.1" iyz="0.0" izz="0.1"/>
         </inertial>
         <visual name="left_wheel_visual">
-           <origin xyz="0.0 0.0 0.0" rpy="0.0 0.0 0.0"/>
-            <geometry>
-                <cylinder radius="0.08" length="0.025"/>
+            <origin xyz="0.0 0.0 0.0" rpy="0.0 0.0 0.0"/>
+            <geometry>
+                <cylinder radius="0.1" length="0.05"/>
             </geometry>
         </visual>
@@ -48,5 +46,5 @@
             <origin xyz="0.0 0.0 0.0" rpy="0.0 0.0 0.0"/>
             <geometry>
-                <cylinder radius="0.08" length="0.025"/>
+                <cylinder radius="0.1" length="0.05"/>
             </geometry>
         </collision>
@@ -55,5 +53,5 @@
         <inertial>
             <origin xyz="0.0 0.0 0.0" rpy="0.0 0.0 0.0"/>
-            <mass value="15.0"/>
+            <mass value="5.0"/>
             <inertia ixx="0.1" ixy="0.0" ixz="0.0" iyy="0.1" iyz="0.0" izz="0.1"/>
         </inertial>
@@ -61,5 +59,5 @@
             <origin xyz="0.0 0.0 0.0" rpy="0.0 0.0 0.0"/>
             <geometry>
-                <cylinder radius="0.08" length="0.025"/>
+                <cylinder radius="0.1" length="0.05"/>
             </geometry>
         </visual>
@@ -67,10 +65,10 @@
             <origin xyz="0.0 0.0 0.0" rpy="0.0 0.0 0.0"/>
             <geometry>
-                <cylinder radius="0.08" length="0.025"/>
+                <cylinder radius="0.1" length="0.05"/>
             </geometry>
         </collision>
     </link>
     <joint name="wheel_left_joint" type="continuous">
-         <origin xyz="0.15 0.20 -0.157" rpy="0.0 1.5705 1.5705"/>
+        <origin xyz="0.0 0.15 0.0" rpy="0.0 1.5705 1.5705"/>
         <parent link="base_link"/>
         <child link="left_wheel"/>
@@ -78,5 +76,5 @@
     </joint>
     <joint name="wheel_right_joint" type="continuous">
-        <origin xyz="0.15 -0.20 -0.157" rpy="0.0 1.5705 1.5705"/>
+        <origin xyz="0.0 -0.15 0.0" rpy="0.0 1.5705 1.5705"/>
         <parent link="base_link"/>
         <child link="right_wheel"/>
@@ -85,12 +83,12 @@
     <link name="front_caster">
         <inertial>
-            <origin xyz="0.0 0.0 0.0" rpy="0.0 1.5707 1.5707"/>
-            <mass value="15.0"/>
-            <inertia ixx="0.1" ixy="0.0" ixz="0.0" iyy="0.1" iyz="0.0" izz="0.1"/>
+            <origin xyz="0.0 0.0 0.0" rpy="0.0 0.0 0.0"/>
+            <mass value="0.0"/>
+            <inertia ixx="0.0" ixy="0.0" ixz="0.0" iyy="0.0" iyz="0.0" izz="0.0"/>
         </inertial>
         <visual name="front_caster_visual">
             <origin xyz="0.0 0.0 0.0" rpy="0.0 0.0 0.0"/>
             <geometry>
-                <cylinder radius="0.08" length="0.025"/>
+                <sphere radius="0.0499"/>
             </geometry>
             <material name="">
@@ -100,25 +98,26 @@
         </visual>
         <collision>
-             <origin xyz="0.0 0.0 0.0" rpy="0.0 0.0 0.0"/>
-            <geometry>
-                <cylinder radius="0.08" length="0.025"/>
+            <origin xyz="0.0 0.0 0.0" rpy="0.0 0.0 0.0"/>
+            <geometry>
+                <sphere radius="0.0499"/>
             </geometry>
         </collision>
     </link>
     <joint name="front_caster_joint" type="fixed">
-        <origin xyz="-0.11 0.275 -0.14" rpy="0.0 1.5705 1.5705"/>
+        <origin xyz="0.15 0.0 -0.05" rpy="0.0 0.0 0.0"/>
         <parent link="base_link"/>
         <child link="front_caster"/>
-    </joint>
-    <link name="back_caster">
-       <inertial>
-            <origin xyz="0.0 0.0 0.0" rpy="0.0 0.0 0.0"/>
-            <mass value="15.0"/>
-            <inertia ixx="0.1" ixy="0.0" ixz="0.0" iyy="0.1" iyz="0.0" izz="0.1"/>
+        <axis xyz="0.0 0.0 0.0"/>
+    </joint>
+ <link name="back_caster">
+        <inertial>
+            <origin xyz="0.0 0.0 0.0" rpy="0.0 0.0 0.0"/>
+            <mass value="0.0"/>
+            <inertia ixx="0.0" ixy="0.0" ixz="0.0" iyy="0.0" iyz="0.0" izz="0.0"/>
         </inertial>
         <visual name="back_caster_visual">
             <origin xyz="0.0 0.0 0.0" rpy="0.0 0.0 0.0"/>
             <geometry>
-                <cylinder radius="0.08" length="0.025"/>
+                <sphere radius="0.0499"/>
             </geometry>
             <material name="">
@@ -128,46 +127,100 @@
         </visual>
         <collision>
-           <origin xyz="0.0 0.0 0.0" rpy="0.0 0.0 0.0"/>
-            <geometry>
-                <cylinder radius="0.08" length="0.025"/>
+            <origin xyz="0.0 0.0 0.0" rpy="0.0 0.0 0.0"/>
+            <geometry>
+                <sphere radius="0.0499"/>
             </geometry>
         </collision>
     </link>
     <joint name="back_caster_joint" type="fixed">
-       <origin xyz="-0.11 -0.275 -0.14" rpy="0.0 1.5705 1.5705"/>
+        <origin xyz="-0.15 0.0 -0.05" rpy="0.0 0.0 0.0"/>
         <parent link="base_link"/>
         <child link="back_caster"/>
+        <axis xyz="0.0 0.0 0.0"/>
+    </joint>
+    <link name="lidar_link">
+        <inertial>
+            <origin xyz="0.0 0.0 0.0" rpy="0.0 0.0 0.0"/>
+            <mass value="0.1"/>
+            <inertia ixx="0.0" ixy="0.0" ixz="0.0" iyy="0.0" iyz="0.0" izz="0.0"/>
+        </inertial>
+        <visual name="lidar_link_visual">
+            <origin xyz="0.0 0.0 0.0" rpy="0.0 0.0 0.0"/>
+            <geometry>
+                <mesh filename="package://diffrobot_description/meshes/lidar_link.STL"/>
+            </geometry>
+            <material name="">
+                <color rgba="1.0 0.0 0.0 1.0"/>
+                <texture filename=""/>
+            </material>
+        </visual>
+        <collision>
+            <origin xyz="0.0 0.0 0.0" rpy="0.0 0.0 0.0"/>
+            <geometry>
+                <box size="0.1 0.1 0.1"/>
+            </geometry>
+        </collision>
+    </link>
+    <joint name="lidar_joint" type="fixed">
+        <origin xyz="0.11 0.0 0.12" rpy="1.5708 0.0 1.5708"/>
+        <parent link="base_link"/>
+        <child link="lidar_link"/>
     </joint>
     <link name="laser">
-        <visual name="laser_visual">
-            <origin xyz="0.0 0.0 0.0" rpy="0.0 0.0 0.0"/>
-            <geometry>
-                <box size="0.05 0.05 0.05"/>
-            </geometry>
-        </visual>
-        <collision name="laser_collision">
-            <origin xyz="0.0 0.0 0.0" rpy="0.0 0.0 0.0"/>
-            <geometry>
-                <box size="0.05 0.05 0.05"/>
-            </geometry>
-        </collision>
     </link>
     <joint name="laser_data_joint" type="fixed">
-        <origin xyz="0.20 0.0 0.13" rpy="0.0 0.0 0.0"/>
-        <parent link="base_link"/>
+        <origin xyz="0.0 0.0 0.0" rpy="0.0 -1.5708 -1.5708"/>
+        <parent link="lidar_link"/>
         <child link="laser"/>
     </joint>
+    <link name="gps_link">
+        <collision>
+        <origin xyz="0 0 0.1" rpy="0 0 0"/>
+        <geometry>
+            <box size="0.02 0.02 0.02"/>
+        </geometry>
+        </collision>
+        <visual>
+        <origin xyz="0 0 0.1" rpy="0 0 0"/>
+        <geometry>
+            <box size="0.02 0.02 0.02"/>
+        </geometry>
+        <material name="orange"/>
+        </visual>
+        <inertial>
+        <origin xyz="0 0 1" rpy="0 0 0"/>
+        <mass value="1"/>
+        <inertia
+            ixx="1.0" ixy="0.0" ixz="0.0"
+            iyy="1.0" iyz="0.0"
+            izz="1.0"/>
+        </inertial>
+    </link>
+    <joint name="gps_joint" type="fixed">
+        <origin xyz="0.0 0.0 0.0" rpy="0.0 0.0 0.0"/>
+        <parent link="base_link"/>
+        <child link="gps_link"/>
+    </joint>
     <link name="imu_link">
+        <collision>
+        <origin xyz="0 0 0.1" rpy="0 0 0"/>
+        <geometry>
+            <box size="0.02 0.02 0.02"/>
+        </geometry>
+        </collision>
         <visual>
-            <origin xyz="0 0 0" rpy="0 0 0"/>
-            <geometry>
-                <box size="0.03 0.1 0.03"/>
-            </geometry>
-            <material name="orange"/> <!-- Add this to fix the material warning -->
-        </visual>
-        <inertial>
-            <origin xyz="0 0 0" rpy="0 0 0"/>
-            <mass value="0.1"/> <!-- Reduced mass (1kg is too heavy for an IMU) -->
-            <inertia ixx="1e-4" ixy="0.0" ixz="0.0" iyy="1e-4" iyz="0.0" izz="1e-4"/>
+        <origin xyz="0 0 0.1" rpy="0 0 0"/>
+        <geometry>
+            <box size="0.02 0.02 0.02"/>
+        </geometry>
+        <material name="orange"/>
+        </visual>
+        <inertial>
+        <origin xyz="0 0 1" rpy="0 0 0"/>
+        <mass value="1"/>
+        <inertia
+            ixx="1.0" ixy="0.0" ixz="0.0"
+            iyy="1.0" iyz="0.0"
+            izz="1.0"/>
         </inertial>
     </link>
