Commit message: updates

File: src/module2/diffrobot_description/urdf/diffrobot.xacro (robot description, xacro)
@@ -1,201 +1,194 @@
 <?xml version='1.0'?>
 <robot name="diffrobot" xmlns:xacro="http://www.ros.org/wiki/xacro">
-  <!-- Materials -->
-  <material name="blue">
-    <color rgba="0.0 0.0 1.0 1.0"/>
-  </material>
-  <material name="white">
-    <color rgba="1.0 1.0 1.0 1.0"/>
-  </material>
-  <material name="orange">
-    <color rgba="1.0 0.5 0.0 1.0"/>
-  </material>
-  <material name="black">
-    <color rgba="0.0 0.0 0.0 1.0"/>
-  </material>
-  <!-- Base Footprint (Reference Frame) -->
-  <link name="base_footprint"/>
-  <!-- Base Link -->
-  <joint name="base_footprint_joint" type="fixed">
-    <parent link="base_footprint"/>
-    <child link="base_link"/>
-  </joint>
-  <link name="base_link">
-    <inertial>
-      <origin xyz="0.0 0.0 0.145" rpy="0.0 0.0 0.0"/>
-      <mass value="15.0"/>
-      <inertia ixx="0.1" ixy="0.0" ixz="0.0" iyy="0.1" iyz="0.0" izz="0.1"/>
-    </inertial>
-    <visual>
-      <origin xyz="0.0 0.0 0.0" rpy="0.0 0.0 0.0"/>
-      <geometry>
-        <box size="0.52 0.52 0.155"/>
-      </geometry>
-      <material name="blue"/>
-    </visual>
-    <collision>
-      <origin xyz="0.0 0.0 0.0" rpy="0.0 0.0 0.0"/>
-      <geometry>
-        <box size="0.52 0.52 0.155"/>
-      </geometry>
-    </collision>
-  </link>
-  <!-- Wheels -->
-  <link name="left_wheel">
-    <inertial>
-      <origin xyz="0.0 0.0 0.0" rpy="0.0 0.0 0.0"/>
-      <mass value="1.0"/>
-      <inertia ixx="0.01" ixy="0.0" ixz="0.0" iyy="0.01" iyz="0.0" izz="0.02"/>
-    </inertial>
-    <visual>
-      <origin xyz="0.0 0.0 0.0" rpy="0.0 1.5708 0.0"/>
-      <geometry>
-        <cylinder radius="0.08" length="0.025"/>
-      </geometry>
-      <material name="black"/>
-    </visual>
-    <collision>
-      <origin xyz="0.0 0.0 0.0" rpy="0.0 1.5708 0.0"/>
-      <geometry>
-        <cylinder radius="0.08" length="0.025"/>
-      </geometry>
-    </collision>
-  </link>
-  <link name="right_wheel">
-    <inertial>
-      <origin xyz="0.0 0.0 0.0" rpy="0.0 0.0 0.0"/>
-      <mass value="1.0"/>
-      <inertia ixx="0.01" ixy="0.0" ixz="0.0" iyy="0.01" iyz="0.0" izz="0.02"/>
-    </inertial>
-    <visual>
-      <origin xyz="0.0 0.0 0.0" rpy="0.0 1.5708 0.0"/>
-      <geometry>
-        <cylinder radius="0.08" length="0.025"/>
-      </geometry>
-      <material name="black"/>
-    </visual>
-    <collision>
-      <origin xyz="0.0 0.0 0.0" rpy="0.0 1.5708 0.0"/>
-      <geometry>
-        <cylinder radius="0.08" length="0.025"/>
-      </geometry>
-    </collision>
-  </link>
-  <!-- Wheel Joints -->
-  <joint name="wheel_left_joint" type="continuous">
-    <origin xyz="0.15 0.20 -0.157" rpy="0.0 0.0 0.0"/>
-    <parent link="base_link"/>
-    <child link="left_wheel"/>
-    <axis xyz="0.0 0.0 1.0"/>
-  </joint>
-  <joint name="wheel_right_joint" type="continuous">
-    <origin xyz="0.15 -0.20 -0.157" rpy="0.0 0.0 0.0"/>
-    <parent link="base_link"/>
-    <child link="right_wheel"/>
-    <axis xyz="0.0 0.0 1.0"/>
-  </joint>
-  <!-- Casters -->
-  <link name="front_caster">
-    <inertial>
-      <origin xyz="0.0 0.0 0.0" rpy="0.0 0.0 0.0"/>
-      <mass value="0.5"/>
-      <inertia ixx="0.001" ixy="0.0" ixz="0.0" iyy="0.001" iyz="0.0" izz="0.001"/>
-    </inertial>
-    <visual>
-      <origin xyz="0.0 0.0 0.0" rpy="0.0 1.5708 0.0"/>
-      <geometry>
-        <cylinder radius="0.08" length="0.025"/>
-      </geometry>
-      <material name="white"/>
-    </visual>
-    <collision>
-      <origin xyz="0.0 0.0 0.0" rpy="0.0 1.5708 0.0"/>
-      <geometry>
-        <cylinder radius="0.08" length="0.025"/>
-      </geometry>
-    </collision>
-  </link>
-  <link name="back_caster">
-    <inertial>
-      <origin xyz="0.0 0.0 0.0" rpy="0.0 0.0 0.0"/>
-      <mass value="0.5"/>
-      <inertia ixx="0.001" ixy="0.0" ixz="0.0" iyy="0.001" iyz="0.0" izz="0.001"/>
-    </inertial>
-    <visual>
-      <origin xyz="0.0 0.0 0.0" rpy="0.0 1.5708 0.0"/>
-      <geometry>
-        <cylinder radius="0.08" length="0.025"/>
-      </geometry>
-      <material name="white"/>
-    </visual>
-    <collision>
-      <origin xyz="0.0 0.0 0.0" rpy="0.0 1.5708 0.0"/>
-      <geometry>
-        <cylinder radius="0.08" length="0.025"/>
-      </geometry>
-    </collision>
-  </link>
-  <!-- Caster Joints -->
-  <joint name="front_caster_joint" type="fixed">
-    <origin xyz="-0.11 0.275 -0.14" rpy="0.0 0.0 0.0"/>
-    <parent link="base_link"/>
-    <child link="front_caster"/>
-  </joint>
-  <joint name="back_caster_joint" type="fixed">
-    <origin xyz="-0.11 -0.275 -0.14" rpy="0.0 0.0 0.0"/>
-    <parent link="base_link"/>
-    <child link="back_caster"/>
-  </joint>
-  <!-- Laser (LIDAR) -->
-  <link name="laser">
-    <inertial>
-      <origin xyz="0.0 0.0 0.0" rpy="0.0 0.0 0.0"/>
-      <mass value="0.1"/>
-      <inertia ixx="0.001" ixy="0.0" ixz="0.0" iyy="0.001" iyz="0.0" izz="0.001"/>
-    </inertial>
-    <visual>
-      <origin xyz="0.0 0.0 0.0" rpy="0.0 0.0 0.0"/>
-      <geometry>
-        <box size="0.05 0.05 0.05"/>
-      </geometry>
-      <material name="orange"/>
-    </visual>
-    <collision>
-      <origin xyz="0.0 0.0 0.0" rpy="0.0 0.0 0.0"/>
-      <geometry>
-        <box size="0.05 0.05 0.05"/>
-      </geometry>
-    </collision>
-  </link>
-  <joint name="laser_joint" type="fixed">
-    <origin xyz="0.20 0.0 0.13" rpy="0.0 0.0 0.0"/>
-    <parent link="base_link"/>
-    <child link="laser"/>
-  </joint>
-  <!-- IMU -->
-  <link name="imu_link">
-    <inertial>
-      <origin xyz="0.0 0.0 0.0" rpy="0.0 0.0 0.0"/>
-      <mass value="0.1"/>
-      <inertia ixx="0.0001" ixy="0.0" ixz="0.0" iyy="0.0001" iyz="0.0" izz="0.0001"/>
-    </inertial>
-    <visual>
-      <origin xyz="0.0 0.0 0.0" rpy="0.0 0.0 0.0"/>
-      <geometry>
-        <box size="0.03 0.1 0.03"/>
-      </geometry>
-      <material name="orange"/>
-    </visual>
-    <collision>
-      <origin xyz="0.0 0.0 0.0" rpy="0.0 0.0 0.0"/>
-      <geometry>
-        <box size="0.03 0.1 0.03"/>
-      </geometry>
-    </collision>
-  </link>
-  <joint name="imu_joint" type="fixed">
-    <origin xyz="0.26 0.0 0.0" rpy="0.0 0.0 0.0"/>
-    <parent link="base_link"/>
-    <child link="imu_link"/>
-  </joint>
+    <xacro:include filename="$(find diffrobot_description)/urdf/diffrobot.gazebo"/>
+    <link name="base_footprint"/>
+    <joint name="robot_footprint_joint" type="fixed">
+        <origin xyz="0 0 0.145" rpy="0 0 0" />
+        <parent link="base_footprint"/>
+        <child link="base_link"/>
+    </joint>
+    <link name="base_link">
+        <inertial>
+            <origin xyz="0.0 0.0 0.0" rpy="0.0 0.0 0.0"/>
+            <mass value="15.0"/>
+            <inertia ixx="0.0" ixy="0.0" ixz="0.0" iyy="0.0" iyz="0.0" izz="0.0"/>
+        </inertial>
+        <visual name="base_link_visual">
+            <origin xyz="0.0 0.0 0.0" rpy="0.0 0.0 0.0"/>
+            <geometry>
+                <box size="0.52 0.52 0.155"/>
+            </geometry>
+            <material name="">
+                <color rgba="0.0 0.0 1.0 1.0"/>
+                <texture filename=""/>
+            </material>
+        </visual>
+        <collision>
+            <origin xyz="0.0 0.0 0.0" rpy="0.0 0.0 0.0"/>
+            <geometry>
+                <box size="0.52 0.52 0.155"/>
+            </geometry>
+        </collision>
+    </link>
+    <link name="left_wheel">
+        <inertial>
+            <origin xyz="0.0 0.0 0.0" rpy="0.0 1.5707 1.5707"/>
+            <mass value="15.0"/>
+            <inertia ixx="0.1" ixy="0.0" ixz="0.0" iyy="0.1" iyz="0.0" izz="0.1"/>
+        </inertial>
+        <visual name="left_wheel_visual">
+            <origin xyz="0.0 0.0 0.0" rpy="0.0 0.0 0.0"/>
+            <geometry>
+                <cylinder radius="0.08" length="0.025"/>
+            </geometry>
+        </visual>
+        <collision name='left_wheel_collision'>
+            <origin xyz="0.0 0.0 0.0" rpy="0.0 0.0 0.0"/>
+            <geometry>
+                <cylinder radius="0.08" length="0.025"/>
+            </geometry>
+        </collision>
+    </link>
+    <link name="right_wheel">
+        <inertial>
+            <origin xyz="0.0 0.0 0.0" rpy="0.0 0.0 0.0"/>
+            <mass value="15.0"/>
+            <inertia ixx="0.1" ixy="0.0" ixz="0.0" iyy="0.1" iyz="0.0" izz="0.1"/>
+        </inertial>
+        <visual name="right_wheel_visual">
+            <origin xyz="0.0 0.0 0.0" rpy="0.0 0.0 0.0"/>
+            <geometry>
+                <cylinder radius="0.08" length="0.025"/>
+            </geometry>
+        </visual>
+        <collision name='right_wheel_collision'>
+            <origin xyz="0.0 0.0 0.0" rpy="0.0 0.0 0.0"/>
+            <geometry>
+                <cylinder radius="0.08" length="0.025"/>
+            </geometry>
+        </collision>
+    </link>
+    <joint name="wheel_left_joint" type="continuous">
+        <origin xyz="0.15 0.20 -0.157" rpy="0.0 1.5705 1.5705"/>
+        <parent link="base_link"/>
+        <child link="left_wheel"/>
+        <axis xyz="0.0 0.0 1.0"/>
+    </joint>
+    <joint name="wheel_right_joint" type="continuous">
+        <origin xyz="0.15 -0.20 -0.157" rpy="0.0 1.5705 1.5705"/>
+        <parent link="base_link"/>
+        <child link="right_wheel"/>
+        <axis xyz="0.0 0.0 1.0"/>
+    </joint>
+    <link name="front_caster">
+        <inertial>
+            <origin xyz="0.0 0.0 0.0" rpy="0.0 0.0 0.0"/>
+            <mass value="15.0"/>
+            <inertia ixx="0.1" ixy="0.0" ixz="0.0" iyy="0.0" iyz="0.0" izz="0.0"/>
+        </inertial>
+        <visual name="front_caster_visual">
+            <origin xyz="0.0 0.0 0.0" rpy="0.0 0.0 0.0"/>
+            <geometry>
+                <cylinder radius="0.08" length="0.025"/>
+            </geometry>
+            <material name="">
+                <color rgba="1.0 1.0 1.0 1.0"/>
+                <texture filename=""/>
+            </material>
+        </visual>
+        <collision>
+            <origin xyz="0.0 0.0 0.0" rpy="0.0 0.0 0.0"/>
+            <geometry>
+                <cylinder radius="0.08" length="0.025"/>
+            </geometry>
+        </collision>
+    </link>
+    <joint name="front_caster_joint" type="fixed">
+        <origin xyz="-0.11 0.275 -0.157" rpy="0.0 1.5705 1.5705"/>
+        <parent link="base_link"/>
+        <child link="front_caster"/>
+        <axis xyz="0.0 0.0 1.0"/>
+    </joint>
+ <link name="back_caster">
+        <inertial>
+            <origin xyz="0.0 0.0 0.0" rpy="0.0 0.0 0.0"/>
+            <mass value="15.0"/>
+            <inertia ixx="0.1" ixy="0.0" ixz="0.0" iyy="0.1" iyz="0.0" izz="0.1"/>
+        </inertial>
+        <visual name="back_caster_visual">
+            <origin xyz="0.0 0.0 0.0" rpy="0.0 0.0 0.0"/>
+            <geometry>
+                <cylinder radius="0.08" length="0.025"/>
+            </geometry>
+            <material name="">
+                <color rgba="1.0 1.0 1.0 1.0"/>
+                <texture filename=""/>
+            </material>
+        </visual>
+        <collision>
+            <origin xyz="0.0 0.0 0.0" rpy="0.0 0.0 0.0"/>
+            <geometry>
+                <cylinder radius="0.08" length="0.025"/>
+            </geometry>
+        </collision>
+    </link>
+    <joint name="back_caster_joint" type="fixed">
+        <origin xyz="-0.11 -0.275 -0.157" rpy="0.0 1.5705 1.5705"/>
+        <parent link="base_link"/>
+        <child link="back_caster"/>
+        <axis xyz="0.0 0.0 0.0"/>
+    </joint>
+    <link name="laser">
+      <inertial>
+        <origin xyz="0.0 0.0 0.0" rpy="0.0 0.0 0.0"/>
+        <mass value="0.1"/>
+        <inertia ixx="0.001" ixy="0.0" ixz="0.0" iyy="0.001" iyz="0.0" izz="0.001"/>
+      </inertial>
+      <visual>
+        <origin xyz="0.0 0.0 0.0" rpy="0.0 0.0 0.0"/>
+        <geometry>
+          <box size="0.05 0.05 0.05"/>
+        </geometry>
+        <material name="orange"/>
+      </visual>
+      <collision>
+        <origin xyz="0.0 0.0 0.0" rpy="0.0 0.0 0.0"/>
+        <geometry>
+          <box size="0.05 0.05 0.05"/>
+        </geometry>
+      </collision>
+    </link>
+    <joint name="laser_joint" type="fixed">
+      <origin xyz="0.20 0.0 0.13" rpy="0.0 0.0 0.0"/>
+      <parent link="base_link"/>
+      <child link="laser"/>
+    </joint>
+     <link name="imu_link">
+        <collision>
+        <origin xyz="0 0 0.1" rpy="0 0 0"/>
+        <geometry>
+            <box size="0.02 0.02 0.02"/>
+        </geometry>
+        </collision>
+        <visual>
+        <origin xyz="0.26 0 0" rpy="0 0 0"/>
+        <geometry>
+             <box size="0.03 0.1 0.03"/>
+        </geometry>
+        <material name="orange"/>
+        </visual>
+        <inertial>
+        <origin xyz="0 0 1" rpy="0 0 0"/>
+        <mass value="1"/>
+        <inertia
+            ixx="1.0" ixy="0.0" ixz="0.0"
+            iyy="1.0" iyz="0.0"
+            izz="1.0"/>
+        </inertial>
+    </link>
+    <joint name="imu_joint" type="fixed">
+        <origin xyz="0.0 0.0 0.0" rpy="0.0 0.0 0.0"/>
+        <parent link="base_link"/>
+        <child link="imu_link"/>
+    </joint>
 </robot>

Commit message: xacro

File: src/module2/diffrobot_description/urdf/diffrobot.xacro (robot description, xacro)
@@ -3,5 +3,5 @@
     <xacro:include filename="$(find diffrobot_description)/urdf/diffrobot.gazebo"/>
     <link name="base_footprint"/>
-    <joint name="robot_footprint_joint" type="fixed">
+    <joint name="base_footprint_joint" type="fixed">
         <origin xyz="0 0 0.145" rpy="0 0 0" />
         <parent link="base_footprint"/>

Commit message: updates

File: src/module2/diffrobot_description/urdf/diffrobot.xacro (robot description, xacro)
@@ -4,5 +4,5 @@
     <link name="base_footprint"/>
     <joint name="base_footprint_joint" type="fixed">
-        <origin xyz="0 0 0.145" rpy="0 0 0" />
+        <!-- <origin xyz="0 0 0.145" rpy="0 0 0" /> -->
         <parent link="base_footprint"/>
         <child link="base_link"/>
@@ -10,5 +10,5 @@
     <link name="base_link">
         <inertial>
-            <origin xyz="0.0 0.0 0.0" rpy="0.0 0.0 0.0"/>
+            <origin xyz="0.0 0.0 0.145" rpy="0.0 0.0 0.0"/>
             <mass value="15.0"/>
             <inertia ixx="0.0" ixy="0.0" ixz="0.0" iyy="0.0" iyz="0.0" izz="0.0"/>

Commit message: update

File: src/module2/diffrobot_description/urdf/diffrobot.xacro (robot description, xacro)
@@ -1,3 +1,234 @@
 <?xml version='1.0'?>
+<robot name="diffrobot" xmlns:xacro="http://www.ros.org/wiki/xacro">
+    <xacro:include filename="$(find diffrobot_description)/urdf/diffrobot.gazebo"/>
+    <link name="base_footprint"/>
+  <joint name="base_footprint_joint" type="fixed">
+      <parent link="base_footprint"/>
+      <child link="base_link"/>
+  </joint>
+    <link name="base_link">
+        <inertial>
+            <origin xyz="0.0 0.0 0.0" rpy="0.0 0.0 0.0"/>
+            <mass value="15.0"/>
+            <inertia ixx="0.0" ixy="0.0" ixz="0.0" iyy="0.0" iyz="0.0" izz="0.0"/>
+        </inertial>
+        <visual name="base_link_visual">
+            <origin xyz="0.0 0.0 0.0" rpy="0.0 0.0 0.0"/>
+            <geometry>
+                <box size="0.52 0.52 0.155"/>
+            </geometry>
+            <material name="">
+                <color rgba="0.0 0.0 1.0 1.0"/>
+                <texture filename=""/>
+            </material>
+        </visual>
+        <collision>
+            <origin xyz="0.0 0.0 0.0" rpy="0.0 0.0 0.0"/>
+            <geometry>
+                <box size="0.52 0.52 0.155"/>
+            </geometry>
+        </collision>
+    </link>
+    <link name="left_wheel">
+       <inertial>
+            <origin xyz="0.0 0.0 0.0" rpy="0.0 0.0 0.0"/>
+            <mass value="15.0"/>
+            <inertia ixx="0.1" ixy="0.0" ixz="0.0" iyy="0.1" iyz="0.0" izz="0.1"/>
+        </inertial>
+        <visual name="left_wheel_visual">
+           <origin xyz="0.0 0.0 0.0" rpy="0.0 0.0 0.0"/>
+            <geometry>
+                <cylinder radius="0.08" length="0.025"/>
+            </geometry>
+        </visual>
+        <collision name='left_wheel_collision'>
+            <origin xyz="0.0 0.0 0.0" rpy="0.0 0.0 0.0"/>
+            <geometry>
+                <cylinder radius="0.08" length="0.025"/>
+            </geometry>
+        </collision>
+    </link>
+    <link name="right_wheel">
+        <inertial>
+            <origin xyz="0.0 0.0 0.0" rpy="0.0 0.0 0.0"/>
+            <mass value="15.0"/>
+            <inertia ixx="0.1" ixy="0.0" ixz="0.0" iyy="0.1" iyz="0.0" izz="0.1"/>
+        </inertial>
+        <visual name="right_wheel_visual">
+            <origin xyz="0.0 0.0 0.0" rpy="0.0 0.0 0.0"/>
+            <geometry>
+                <cylinder radius="0.08" length="0.025"/>
+            </geometry>
+        </visual>
+        <collision name='right_wheel_collision'>
+            <origin xyz="0.0 0.0 0.0" rpy="0.0 0.0 0.0"/>
+            <geometry>
+                <cylinder radius="0.08" length="0.025"/>
+            </geometry>
+        </collision>
+    </link>
+    <joint name="wheel_left_joint" type="continuous">
+         <origin xyz="0.15 0.20 -0.157" rpy="0.0 1.5705 1.5705"/>
+        <parent link="base_link"/>
+        <child link="left_wheel"/>
+        <axis xyz="0.0 0.0 1.0"/>
+    </joint>
+    <joint name="wheel_right_joint" type="continuous">
+        <origin xyz="0.15 -0.20 -0.157" rpy="0.0 1.5705 1.5705"/>
+        <parent link="base_link"/>
+        <child link="right_wheel"/>
+        <axis xyz="0.0 0.0 1.0"/>
+    </joint>
+    <link name="front_caster">
+        <inertial>
+            <origin xyz="0.0 0.0 0.0" rpy="0.0 1.5707 1.5707"/>
+            <mass value="15.0"/>
+            <inertia ixx="0.1" ixy="0.0" ixz="0.0" iyy="0.1" iyz="0.0" izz="0.1"/>
+        </inertial>
+        <visual name="front_caster_visual">
+            <origin xyz="0.0 0.0 0.0" rpy="0.0 0.0 0.0"/>
+            <geometry>
+                <cylinder radius="0.0625" length="0.025"/>
+            </geometry>
+            <material name="">
+                <color rgba="1.0 1.0 1.0 1.0"/>
+                <texture filename=""/>
+            </material>
+        </visual>
+        <collision>
+             <origin xyz="0.0 0.0 0.0" rpy="0.0 0.0 0.0"/>
+            <geometry>
+                <cylinder radius="0.0625" length="0.025"/>
+            </geometry>
+        </collision>
+    </link>
+    <joint name="front_caster_joint" type="fixed">
+        <origin xyz="-0.11 0.275 -0.14" rpy="0.0 1.5705 1.5705"/>
+        <parent link="base_link"/>
+        <child link="front_caster"/>
+        <axis xyz="0.0 0.0 1.0"/>
+    </joint>
+ <link name="back_caster">
+       <inertial>
+            <origin xyz="0.0 0.0 0.0" rpy="0.0 0.0 0.0"/>
+            <mass value="15.0"/>
+            <inertia ixx="0.1" ixy="0.0" ixz="0.0" iyy="0.1" iyz="0.0" izz="0.1"/>
+        </inertial>
+        <visual name="back_caster_visual">
+            <origin xyz="0.0 0.0 0.0" rpy="0.0 0.0 0.0"/>
+            <geometry>
+                <cylinder radius="0.0625" length="0.025"/>
+            </geometry>
+            <material name="">
+                <color rgba="1.0 1.0 1.0 1.0"/>
+                <texture filename=""/>
+            </material>
+        </visual>
+        <collision>
+           <origin xyz="0.0 0.0 0.0" rpy="0.0 0.0 0.0"/>
+            <geometry>
+                <cylinder radius="0.0625" length="0.025"/>
+            </geometry>
+        </collision>
+    </link>
+    <joint name="back_caster_joint" type="fixed">
+       <origin xyz="-0.11 -0.275 -0.14" rpy="0.0 1.5705 1.5705"/>
+        <parent link="base_link"/>
+        <child link="back_caster"/>
+        <axis xyz="0.0 0.0 0.0"/>
+    </joint>
+    <link name="lidar_link">
+        <inertial>
+            <origin xyz="0.0 0.0 0.0" rpy="0.0 0.0 0.0"/>
+            <mass value="0.1"/>
+            <inertia ixx="0.0" ixy="0.0" ixz="0.0" iyy="0.0" iyz="0.0" izz="0.0"/>
+        </inertial>
+        <visual name="lidar_link_visual">
+            <origin xyz="0.0 0.0 0.0" rpy="0.0 0.0 0.0"/>
+            <geometry>
+                <mesh filename="package://diffrobot_description/meshes/lidar_link.STL"/>
+            </geometry>
+            <material name="">
+                <color rgba="1.0 0.0 0.0 1.0"/>
+                <texture filename=""/>
+            </material>
+        </visual>
+        <collision>
+            <origin xyz="0.0 0.0 0.0" rpy="0.0 0.0 0.0"/>
+            <geometry>
+                <box size="0.1 0.1 0.1"/>
+            </geometry>
+        </collision>
+    </link>
+    <joint name="lidar_joint" type="fixed">
+       <origin xyz="0.20 0.0 0.13" rpy="0.0 0.0 0.0"/>
+        <parent link="base_link"/>
+        <child link="lidar_link"/>
+    </joint>
+    <link name="laser">
+    </link>
+    <joint name="laser_data_joint" type="fixed">
+        <origin xyz="0.0 0.0 0.0" rpy="0.0 -1.5708 -1.5708"/>
+        <parent link="lidar_link"/>
+        <child link="laser"/>
+    </joint>
+    <link name="gps_link">
+        <collision>
+        <origin xyz="0 0 0.1" rpy="0 0 0"/>
+        <geometry>
+            <box size="0.02 0.02 0.02"/>
+        </geometry>
+        </collision>
+        <visual>
+        <origin xyz="0 0 0.1" rpy="0 0 0"/>
+        <geometry>
+            <box size="0.02 0.02 0.02"/>
+        </geometry>
+        <material name="orange"/>
+        </visual>
+        <inertial>
+        <origin xyz="0 0 1" rpy="0 0 0"/>
+        <mass value="1"/>
+        <inertia
+            ixx="1.0" ixy="0.0" ixz="0.0"
+            iyy="1.0" iyz="0.0"
+            izz="1.0"/>
+        </inertial>
+    </link>
+    <joint name="gps_joint" type="fixed">
+        <origin xyz="0.0 0.0 0.0" rpy="0.0 0.0 0.0"/>
+        <parent link="base_link"/>
+        <child link="gps_link"/>
+    </joint>
+    <link name="imu_link">
+        <collision>
+        <origin xyz="0 0 0.1" rpy="0 0 0"/>
+        <geometry>
+            <box size="0.02 0.02 0.02"/>
+        </geometry>
+        </collision>
+        <visual>
+        <origin xyz="0.26 0 0" rpy="0 0 0"/>
+        <geometry>
+             <box size="0.03 0.1 0.03"/>
+        </geometry>
+        <material name="orange"/>
+        </visual>
+        <inertial>
+        <origin xyz="0 0 1" rpy="0 0 0"/>
+        <mass value="1"/>
+        <inertia
+            ixx="1.0" ixy="0.0" ixz="0.0"
+            iyy="1.0" iyz="0.0"
+            izz="1.0"/>
+        </inertial>
+    </link>
+    <joint name="imu_joint" type="fixed">
+        <origin xyz="0.0 0.0 0.0" rpy="0.0 0.0 0.0"/>
+        <parent link="base_link"/>
+        <child link="imu_link"/>
+    </joint>
+</robot>
+<!-- <?xml version='1.0'?>
 <robot name="diffrobot" xmlns:xacro="http://www.ros.org/wiki/xacro">
     <xacro:include filename="$(find diffrobot_description)/urdf/diffrobot.gazebo"/>
@@ -192,3 +423,3 @@
         <child link="imu_link"/>
     </joint>
-</robot>
+</robot> -->
